File: schematic/Raspi Power.sch (EAGLE design)
At the start: 10 parts, among them K1 G5L, T1 BC237

Commit message: Updated Schematic and configured gitignore
Parts:
- removed C1: 470u, capacitor-wima:C2.5/2
Connections:
- net 3V3: no longer C1.1
- net N$5: no longer C1.2
Changed lines of the file:
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@@
 <?xml version="1.0" encoding="utf-8"?>
 <!DOCTYPE eagle SYSTEM "eagle.dtd">
-<eagle version="8.0.2">
+<eagle version="8.2.1">
 <drawing>
 <settings>
@@
 <part name="R2" library="resistor" deviceset="R-US_" device="0204/7" value="1K"/>
 <part name="R3" library="resistor" deviceset="R-US_" device="0204/7" value="10K"/>
-<part name="C1" library="capacitor-wima" deviceset="C" device="2.5/2" value="470u"/>
 <part name="IN" library="con-amp-quick" deviceset="M02" device=""/>
 <part name="SL2" library="con-amp-quick" deviceset="M02" device=""/>
@@
 <instance part="R2" gate="G$1" x="71.12" y="20.32" rot="R180"/>
 <instance part="R3" gate="G$1" x="60.96" y="12.7" rot="R90"/>
-<instance part="C1" gate="G$1" x="73.66" y="35.56"/>
 <instance part="IN" gate="G$1" x="5.08" y="73.66"/>
 <instance part="SL2" gate="G$1" x="71.12" y="63.5" rot="R180"/>
@@
 <segment>
 <label x="45.72" y="35.56" size="1.778" layer="95"/>
-<pinref part="C1" gate="G$1" pin="1"/>
-<wire x1="50.8" y1="35.56" x2="48.26" y2="35.56" width="0.1524" layer="91"/>
-<wire x1="73.66" y1="38.1" x2="73.66" y2="45.72" width="0.1524" layer="91"/>
-<wire x1="73.66" y1="45.72" x2="50.8" y2="45.72" width="0.1524" layer="91"/>
-<wire x1="50.8" y1="45.72" x2="50.8" y2="35.56" width="0.1524" layer="91"/>
-<wire x1="50.8" y1="35.56" x2="53.34" y2="35.56" width="0.1524" layer="91"/>
+<wire x1="48.26" y1="35.56" x2="53.34" y2="35.56" width="0.1524" layer="91"/>
 <wire x1="53.34" y1="35.56" x2="53.34" y2="43.18" width="0.1524" layer="91"/>
-<junction x="50.8" y="35.56"/>
 <wire x1="53.34" y1="43.18" x2="63.5" y2="43.18" width="0.1524" layer="91"/>
 <pinref part="S1" gate="B" pin="S"/>
@@
 <wire x1="48.26" y1="20.32" x2="48.26" y2="27.94" width="0.1524" layer="91"/>
 <junction x="60.96" y="20.32"/>
-<pinref part="C1" gate="G$1" pin="2"/>
-<wire x1="73.66" y1="30.48" x2="73.66" y2="25.4" width="0.1524" layer="91"/>
-<wire x1="73.66" y1="25.4" x2="60.96" y2="25.4" width="0.1524" layer="91"/>
-<wire x1="60.96" y1="25.4" x2="60.96" y2="20.32" width="0.1524" layer="91"/>
 <wire x1="48.26" y1="27.94" x2="60.96" y2="27.94" width="0.1524" layer="91"/>
 <pinref part="S1" gate="B" pin="P"/>

Commit message: Fixed initial schematic
Connections:
- net C renamed N$1
- removed net GND: R3.1
- net GNDA: now also R3.1
Other:
- moved on the sheet: IN, K1, R1, R2, R3, S1, SL2, SV1, T1

Commit message: New board design
Parts:
- removed S1: (no value), switch:A68-A31
- removed SV1: (no value), con-lstb:MA03-1
- added JP1, JP2: (no value), pinhead:PINHD-1X2
- added JP3: (no value), pinhead:PINHD-1X3
Connections:
- net 3V3: now also JP2.1, JP3.3; no longer S1B.S, SV1.3
- net 5V-IN: now also JP1.1; no longer S1A.O
- net 5V-OUT: now also JP1.2; no longer S1A.P
- net GPIO-ON: now also JP3.1; no longer SV1.1
- net GPIO-SHTDWN: now also JP3.2; no longer SV1.2
- net N$5: now also JP2.2; no longer S1B.P
Changed lines of the file:
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@@
 <layer number="48" name="Document" color="7" fill="1" visible="no" active="no"/>
 <layer number="49" name="Reference" color="7" fill="1" visible="no" active="no"/>
-<layer number="51" name="tDocu" color="6" fill="1" visible="no" active="no"/>
+<layer number="51" name="tDocu" color="7" fill="1" visible="no" active="no"/>
 <layer number="52" name="bDocu" color="7" fill="1" visible="no" active="no"/>
 <layer number="90" name="Modules" color="5" fill="1" visible="yes" active="yes"/>
@@
 </variantdefs>
 <classes>
-<class number="0" name="default" width="0.6096" drill="0.6096">
-<clearance class="0" value="0.4064"/>
+<class number="0" name="default" width="0.8128" drill="0.6096">
+</class>
+<class number="1" name="ground" width="1.27" drill="1.27">
+</class>
+<class number="2" name="5v" width="1.27" drill="1.27">
+</class>
+<class number="3" name="signal" width="0.8128" drill="0.6096">
+<clearance class="3" value="0.6096"/>
 </class>
 </classes>
@@
 <part name="T1" library="transistor" deviceset="BC237" device=""/>
 <part name="GND2" library="supply1" deviceset="GNDA" device=""/>
-<part name="S1" library="switch" deviceset="A68-A31" device=""/>
 <part name="GND3" library="supply1" deviceset="GNDA" device=""/>
 <part name="R2" library="resistor" deviceset="R-US_" device="0204/7" value="1K"/>
@@
 <part name="SL2" library="con-amp-quick" deviceset="M02" device=""/>
 <part name="GND1" library="supply1" deviceset="GNDA" device=""/>
-<part name="SV1" library="con-lstb" deviceset="MA03-1" device=""/>
 <part name="GND4" library="supply1" deviceset="GNDA" device=""/>
+<part name="JP1" library="pinhead" library_urn="urn:adsk.eagle:library:325" deviceset="PINHD-1X2" device=""/>
+<part name="JP2" library="pinhead" library_urn="urn:adsk.eagle:library:325" deviceset="PINHD-1X2" device=""/>
+<part name="JP3" library="pinhead" library_urn="urn:adsk.eagle:library:325" deviceset="PINHD-1X3" device=""/>
 </parts>
 <sheets>
@@
 <instance part="T1" gate="G$1" x="45.72" y="53.34" rot="R90"/>
 <instance part="GND2" gate="1" x="76.2" y="55.88"/>
-<instance part="S1" gate="B" x="73.66" y="40.64"/>
-<instance part="S1" gate="A" x="48.26" y="81.28"/>
 <instance part="GND3" gate="1" x="25.4" y="66.04"/>
 <instance part="R2" gate="G$1" x="83.82" y="25.4" rot="R180"/>
@@
 <instance part="SL2" gate="G$1" x="83.82" y="68.58" rot="R180"/>
 <instance part="GND1" gate="1" x="53.34" y="22.86"/>
-<instance part="SV1" gate="G$1" x="27.94" y="15.24" rot="R90"/>
 <instance part="GND4" gate="1" x="73.66" y="5.08"/>
+<instance part="JP1" gate="G$1" x="48.26" y="83.82"/>
+<instance part="JP2" gate="G$1" x="86.36" y="45.72"/>
+<instance part="JP3" gate="A" x="27.94" y="15.24" rot="R270"/>
 </instances>
 <busses>
@@
 </segment>
 </net>
-<net name="GNDA" class="0">
+<net name="GNDA" class="1">
 <segment>
 <pinref part="GND2" gate="1" pin="GNDA"/>
@@
 </segment>
 </net>
-<net name="5V-IN" class="0">
+<net name="5V-IN" class="2">
 <segment>
 <wire x1="25.4" y1="81.28" x2="27.94" y2="81.28" width="0.1524" layer="91"/>
@@
 <wire x1="27.94" y1="60.96" x2="38.1" y2="60.96" width="0.1524" layer="91"/>
 <wire x1="27.94" y1="81.28" x2="35.56" y2="81.28" width="0.1524" layer="91"/>
-<wire x1="35.56" y1="81.28" x2="35.56" y2="91.44" width="0.1524" layer="91"/>
+<wire x1="35.56" y1="81.28" x2="35.56" y2="86.36" width="0.1524" layer="91"/>
 <junction x="27.94" y="81.28"/>
 <label x="22.86" y="83.82" size="1.778" layer="95"/>
 <pinref part="K1" gate="2" pin="P"/>
 <pinref part="IN" gate="G$1" pin="2"/>
-<wire x1="35.56" y1="91.44" x2="48.26" y2="91.44" width="0.1524" layer="91"/>
-<pinref part="S1" gate="A" pin="O"/>
-<wire x1="48.26" y1="91.44" x2="48.26" y2="86.36" width="0.1524" layer="91"/>
+<pinref part="JP1" gate="G$1" pin="1"/>
+<wire x1="35.56" y1="86.36" x2="45.72" y2="86.36" width="0.1524" layer="91"/>
 </segment>
 </net>
@@
 <wire x1="45.72" y1="27.94" x2="30.48" y2="27.94" width="0.1524" layer="91"/>
 <label x="33.02" y="27.94" size="1.778" layer="95"/>
-<pinref part="SV1" gate="G$1" pin="1"/>
-<wire x1="30.48" y1="27.94" x2="30.48" y2="22.86" width="0.1524" layer="91"/>
+<pinref part="JP3" gate="A" pin="1"/>
+<wire x1="30.48" y1="27.94" x2="30.48" y2="17.78" width="0.1524" layer="91"/>
 </segment>
 </net>
@@
 </segment>
 <segment>
-<pinref part="SV1" gate="G$1" pin="2"/>
-<wire x1="27.94" y1="22.86" x2="27.94" y2="33.02" width="0.1524" layer="91"/>
 <wire x1="27.94" y1="33.02" x2="17.78" y2="33.02" width="0.1524" layer="91"/>
 <wire x1="17.78" y1="33.02" x2="17.78" y2="38.1" width="0.1524" layer="91"/>
 <wire x1="17.78" y1="38.1" x2="22.86" y2="38.1" width="0.1524" layer="91"/>
 <label x="22.86" y="38.1" size="1.778" layer="95"/>
+<pinref part="JP3" gate="A" pin="2"/>
+<wire x1="27.94" y1="33.02" x2="27.94" y2="17.78" width="0.1524" layer="91"/>
 </segment>
 </net>
@@
 <wire x1="60.96" y1="40.64" x2="66.04" y2="40.64" width="0.1524" layer="91"/>
 <wire x1="66.04" y1="40.64" x2="66.04" y2="48.26" width="0.1524" layer="91"/>
-<wire x1="66.04" y1="48.26" x2="76.2" y2="48.26" width="0.1524" layer="91"/>
-<pinref part="S1" gate="B" pin="S"/>
-<wire x1="76.2" y1="48.26" x2="76.2" y2="45.72" width="0.1524" layer="91"/>
-</segment>
-<segment>
-<pinref part="SV1" gate="G$1" pin="3"/>
-<wire x1="25.4" y1="22.86" x2="25.4" y2="27.94" width="0.1524" layer="91"/>
+<wire x1="66.04" y1="48.26" x2="83.82" y2="48.26" width="0.1524" layer="91"/>
+<pinref part="JP2" gate="G$1" pin="1"/>
+</segment>
+<segment>
 <wire x1="25.4" y1="27.94" x2="15.24" y2="27.94" width="0.1524" layer="91"/>
-<wire x1="15.24" y1="27.94" x2="15.24" y2="40.64" width="0.1524" layer="91"/>
-<wire x1="15.24" y1="40.64" x2="15.24" y2="43.18" width="0.1524" layer="91"/>
+<wire x1="15.24" y1="27.94" x2="15.24" y2="43.18" width="0.1524" layer="91"/>
 <wire x1="15.24" y1="43.18" x2="25.4" y2="43.18" width="0.1524" layer="91"/>
 <label x="25.4" y="43.18" size="1.778" layer="95"/>
+<pinref part="JP3" gate="A" pin="3"/>
+<wire x1="25.4" y1="27.94" x2="25.4" y2="17.78" width="0.1524" layer="91"/>
 </segment>
 </net>
@@
 <wire x1="73.66" y1="22.86" x2="73.66" y2="25.4" width="0.1524" layer="91"/>
 <pinref part="R2" gate="G$1" pin="2"/>
-<wire x1="73.66" y1="25.4" x2="78.74" y2="25.4" width="0.1524" layer="91"/>
-<wire x1="73.66" y1="25.4" x2="73.66" y2="35.56" width="0.1524" layer="91"/>
-<junction x="73.66" y="25.4"/>
-<pinref part="S1" gate="B" pin="P"/>
-</segment>
-</net>
-<net name="5V-OUT" class="0">
+<wire x1="73.66" y1="25.4" x2="76.2" y2="25.4" width="0.1524" layer="91"/>
+<wire x1="76.2" y1="25.4" x2="78.74" y2="25.4" width="0.1524" layer="91"/>
+<wire x1="76.2" y1="25.4" x2="76.2" y2="45.72" width="0.1524" layer="91"/>
+<pinref part="JP2" gate="G$1" pin="2"/>
+<wire x1="76.2" y1="45.72" x2="83.82" y2="45.72" width="0.1524" layer="91"/>
+<junction x="76.2" y="25.4"/>
+</segment>
+</net>
+<net name="5V-OUT" class="2">
 <segment>
 <wire x1="43.18" y1="68.58" x2="50.8" y2="68.58" width="0.1524" layer="91"/>
@@
 <wire x1="60.96" y1="96.52" x2="60.96" y2="68.58" width="0.1524" layer="91"/>
 <junction x="60.96" y="68.58"/>
-<pinref part="S1" gate="A" pin="P"/>
-<wire x1="50.8" y1="68.58" x2="50.8" y2="76.2" width="0.1524" layer="91"/>
-<junction x="50.8" y="68.58"/>
 <pinref part="K1" gate="1" pin="1"/>
 <wire x1="60.96" y1="96.52" x2="53.34" y2="96.52" width="0.1524" layer="91"/>
+<wire x1="50.8" y1="68.58" x2="50.8" y2="76.2" width="0.1524" layer="91"/>
+<wire x1="50.8" y1="76.2" x2="38.1" y2="76.2" width="0.1524" layer="91"/>
+<pinref part="JP1" gate="G$1" pin="2"/>
+<wire x1="38.1" y1="76.2" x2="38.1" y2="83.82" width="0.1524" layer="91"/>
+<wire x1="38.1" y1="83.82" x2="45.72" y2="83.82" width="0.1524" layer="91"/>
+<junction x="50.8" y="68.58"/>
 </segment>
 </net>
@@
 </schematic>
 </drawing>
+<compatibility>
+<note version="8.2" severity="warning">
+Since Version 8.2, Eagle supports online libraries. The ids
+of those online libraries will not be understood (or retained)
+with this version.
+</note>
+</compatibility>
 </eagle>
